Commit message: Add description, gazebo, and nav2 packages with camera, configurable world, and nav2 stack

File: ros2/src/openamrobot_description/urdf/gazebo_control.xacro (robot description, xacro)
@@ -125,4 +125,33 @@
   <xacro:caster_gazebo prefix="bl" />
   <xacro:caster_gazebo prefix="br" />
+  <!-- ── Link-level: camera_link — forward-facing RGB camera ──────── -->
+  <gazebo reference="camera_link">
+    <material>Gazebo/Black</material>
+    <sensor name="camera_sensor" type="camera">
+      <pose relative_to="camera_link">0 0 0 0 0 0</pose>
+      <topic>/rgb_image</topic>
+      <gz_frame_id>camera_optical_frame</gz_frame_id>
+      <update_rate>30</update_rate>
+      <camera>
+        <horizontal_fov>1.047</horizontal_fov>
+        <image>
+          <width>640</width>
+          <height>480</height>
+          <format>R8G8B8</format>
+        </image>
+        <clip>
+          <near>0.05</near>
+          <far>15.0</far>
+        </clip>
+        <noise>
+          <type>gaussian</type>
+          <mean>0.0</mean>
+          <stddev>0.005</stddev>
+        </noise>
+      </camera>
+      <always_on>true</always_on>
+      <visualize>false</visualize>
+    </sensor>
+  </gazebo>
   <!-- ── Link-level: lidar_link — sensor ONLY here ─────────────────── -->
   <gazebo reference="lidar_link">

File: ros2/src/openamrobot_description/urdf/robo_urdf.urdf.xacro (robot description, xacro)
@@ -621,4 +621,38 @@
       xyz="0 0 0" />
   </joint>
+  <!-- Camera link — mounted at front of robot, facing forward -->
+  <link name="camera_link">
+    <visual>
+      <origin xyz="0 0 0" rpy="0 0 0"/>
+      <geometry>
+        <box size="0.04 0.08 0.04"/>
+      </geometry>
+      <material name="camera_black">
+        <color rgba="0.1 0.1 0.1 1"/>
+      </material>
+    </visual>
+    <collision>
+      <origin xyz="0 0 0" rpy="0 0 0"/>
+      <geometry>
+        <box size="0.04 0.08 0.04"/>
+      </geometry>
+    </collision>
+    <inertial>
+      <mass value="0.05"/>
+      <inertia ixx="0.0001" ixy="0" ixz="0" iyy="0.0001" iyz="0" izz="0.0001"/>
+    </inertial>
+  </link>
+  <joint name="camera_joint" type="fixed">
+    <origin xyz="0.35 0 0.20" rpy="0 0 0"/>
+    <parent link="base_link"/>
+    <child link="camera_link"/>
+  </joint>
+  <!-- Optical frame: ROS convention (Z forward, X right, Y down) -->
+  <link name="camera_optical_frame"/>
+  <joint name="camera_optical_joint" type="fixed">
+    <origin xyz="0 0 0" rpy="-1.5707963 0 -1.5707963"/>
+    <parent link="camera_link"/>
+    <child link="camera_optical_frame"/>
+  </joint>
   <xacro:include filename="gazebo_control.xacro" />
 </robot>
